File: harite.kicad_pcb (KiCad board)
At the start: 2 copper layers, 258.2 x 91.6 mm, 76 parts, among them J1 Cirque Connector, J2 Cirque Connector, U1 RP2040_Zero, U2 RP2040_Zero

Commit message: Track cleanup
Routing:
- net RRow 3: track 207.3 -> 204.1 mm
- net RCol 1: track 147.3 -> 144.5 mm
- net RRow 4: track 187.6 -> 185.0 mm
- net RRow 2: track 194.9 -> 192.8 mm
- net RCol 2: track 118.4 -> 116.6 mm

Commit message: Track cleanup
Routing:
- net RRow 1: track 189.2 -> 190.2 mm

Commit message: Add logo
Parts:
- added G***: LOGO, footprints:logo-right, F.Cu at (175.7, 115.1)
- added G***: LOGO, footprints:logo-left, F.Cu at (121.5, 115.1)
